Commit message: making legs

File: connected_bot.urdf (robot description, URDF)
Before this commit: robot leg_design_simplified, 13 links, 8 joints
Links:
- added link fibula_top_left, mass 0.017; collision mesh filename=body_parts/leg_front_left/Body_assemb - Leg_assembly_top_le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; visual mesh filename=body_parts/leg_front_left/Body_assemb - Leg_assembly_top_le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
- link fibula_top_right: geometry collision mesh filename=body_parts/leg_front_right/Body_assemb - Leg_assembly_top_r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; visual mesh filename=body_parts/leg_front_right/Body_assemb - Leg_assembly_top_r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
- link large_link_top_right: geometry collision mesh filename=body_parts/leg_front_right/Body_assemb - Leg_assembly_top_r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; visual mesh filename=body_parts/leg_front_right/Body_assemb - Leg_assembly_top_r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
- link small_link_top_right: geometry collision mesh filename=body_parts/leg_front_right/Body_assemb - Leg_assembly_top_r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; visual mesh filename=body_parts/leg_front_right/Body_assemb - Leg_assembly_top_r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
- link tibia_top_right: geometry collision mesh filename=body_parts/leg_front_right/Body_assemb - Leg_assembly_top_r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; visual mesh filename=body_parts/leg_front_right/Body_assemb - Leg_assembly_top_r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

Commit message: Servo horn extensions all in right place

File: connected_bot.urdf (robot description, URDF)
Before this commit: robot leg_design_simplified, 14 links, 8 joints
Links:
- added link fibula_down_left, mass 0.017; collision mesh filename=body_parts\leg_back_left\Body_assemb - leg_assembly_bottom_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; visual mesh filename=body_parts\leg_back_left\Body_assemb - leg_assembly_bottom_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
- added link fibula_down_right, mass 0.017; collision mesh filename=body_parts\leg_back_right\Body_assemb - Leg_assembly_bottom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; visual mesh filename=body_parts\leg_back_right\Body_assemb - Leg_assembly_bottom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
- added link large_link_down_left, mass 0.017; collision mesh filename=body_parts\leg_back_left\Body_assemb - leg_assembly_bottom_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; visual mesh filename=body_parts\leg_back_left\Body_assemb - leg_assembly_bottom_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
- added link large_link_down_right, mass 0.017; collision mesh filename=body_parts\leg_back_right\Body_assemb - Leg_assembly_bottom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; visual mesh filename=body_parts\leg_back_right\Body_assemb - Leg_assembly_bottom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
- added link large_link_top_left, mass 0.017; collision mesh filename=body_parts\leg_front_left\Body_assemb - Leg_assembly_top_le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; visual mesh filename=body_parts\leg_front_left\Body_assemb - Leg_assembly_top_le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
- added link servo_extension_horn_mock_2_down_left, mass 0.005; collision mesh filename=body_parts\leg_back_left\serve_extent_6.stl; visual mesh filename=body_parts\leg_back_left\serve_extent_6.stl
- added link servo_extension_horn_mock_2_down_right, mass 0.005; collision mesh filename=body_parts\leg_back_right\serve_extent_5.stl; visual mesh filename=body_parts\leg_back_right\serve_extent_5.stl
- added link servo_extension_horn_mock_2_top_left, mass 0.005; collision mesh filename=body_parts\leg_front_left\serve_extent_2.stl; visual mesh filename=body_parts\leg_front_left\serve_extent_2.stl
- added link small_link_down_left, mass 0.002; collision mesh filename=body_parts\leg_back_left\Body_assemb - leg_assembly_bottom_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; visual mesh filename=body_parts\leg_back_left\Body_assemb - leg_assembly_bottom_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
- added link small_link_down_rigth, mass 0.002; collision mesh filename=body_parts\leg_back_right\Body_assemb - Leg_assembly_bottom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; visual mesh filename=body_parts\leg_back_right\Body_assemb - Leg_assembly_bottom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
- added link small_link_top_left, mass 0.002; collision mesh filename=body_parts\leg_front_left\Body_assemb - Leg_assembly_top_le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; visual mesh filename=body_parts\leg_front_left\Body_assemb - Leg_assembly_top_le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
- added link tibia_down_left, mass 0.017; collision mesh filename=body_parts\leg_back_left\Body_assemb - leg_assembly_bottom_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; visual mesh filename=body_parts\leg_back_left\Body_assemb - leg_assembly_bottom_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
- added link tibia_down_right, mass 0.017; collision mesh filename=body_parts\leg_back_right\Body_assemb - Leg_assembly_bottom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; visual mesh filename=body_parts\leg_back_right\Body_assemb - Leg_assembly_bottom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
- added link tibia_top_left, mass 0.017; collision mesh filename=body_parts\leg_front_left\Body_assemb - Leg_assembly_top_le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; visual mesh filename=body_parts\leg_front_left\Body_assemb - Leg_assembly_top_le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
- link servo_extension_horn_mock_2_top_right: geometry collision mesh filename=body_parts\leg_front_right\serve_extent.stl; visual mesh filename=body_parts\leg_front_right\serve_extent.stl

Commit message: Update URDF: Adjust inertial properties and add new servo extension links and joints

File: connected_bot.urdf (robot description, URDF)
Before this commit: robot leg_design_simplified, 28 links, 8 joints
Links:
- added link servo_extension_horn_mock_1_back_left, mass 0.005; collision mesh filename=body_parts\leg_back_left\serve_extent_8.stl; visual mesh filename=body_parts\leg_back_left\serve_extent_8.stl
- added link servo_extension_horn_mock_1_back_right, mass 0.005; collision mesh filename=body_parts\leg_back_right\serve_extent_7.stl; visual mesh filename=body_parts\leg_back_right\serve_extent_7.stl
- added link servo_extension_horn_mock_1_top_left, mass 0.005; collision mesh filename=body_parts\leg_front_left\serve_extent_4.stl; visual mesh filename=body_parts\leg_front_left\serve_extent_4.stl
- link servo_extension_horn_mock_1_top_right: geometry collision mesh filename=body_parts\leg_front_right\serve_extent_3.stl; visual mesh filename=body_parts\leg_front_right\serve_extent_3.stl
Joints:
- added joint fibula_on_hip_down_left: type revolute, parent hip_down_left, child fibula_down_left, origin xyz=0 0 0 rpy=0 0 0, axis 1 0 0, limit effort=0 velocity=0
- added joint fibula_on_hip_down_right: type revolute, parent hip_down_right, child fibula_down_right, origin xyz=0 0 0 rpy=0 0 0, axis 1 0 0, limit effort=0 velocity=0
- added joint fibula_on_hip_top_left: type revolute, parent hip_top_left, child fibula_top_left, origin xyz=0 0 0 rpy=0 0 0, axis 1 0 0, limit effort=0 velocity=0
- added joint fibula_on_hip_top_right: type revolute, parent hip_top_right, child fibula_top_right, origin xyz=0 0 0 rpy=0 0 0, axis 0 1 0, limit lower=0 upper=1 effort=100 velocity=0
- added joint hip_down_left_on_body: type revolute, parent body, child hip_down_left, origin xyz=0 0 0 rpy=0 0 0
- added joint hip_down_right_on_body: type revolute, parent body, child hip_down_right, origin xyz=0 0 0 rpy=0 0 0
- added joint hip_top_left_on_body: type revolute, parent body, child hip_top_left, origin xyz=0 0 0 rpy=0 0 0, axis 0 1 0, limit lower=0 upper=1 effort=100 velocity=100
- added joint hip_top_right_on_body: type revolute, parent body, child hip_top_right, origin xyz=0 0 0 rpy=0 0 0, axis 1 0 0, limit lower=0 upper=1 effort=1 velocity=1

Commit message: Update URDF: Replace mesh origins and adjust joint parameters for new body parts

File: connected_bot.urdf (robot description, URDF)
Before this commit: robot leg_design_simplified, 31 links, 16 joints
Links:
- link body: geometry collision mesh filename=new_body_parts\V0Body_assemb_-_Mirrored_Body_Skeleton_Botto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; visual mesh filename=new_body_parts\V0Body_assemb_-_Mirrored_Body_Skeleton_Botto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
- link fibula_down_right: geometry collision mesh filename=body_parts\leg_back_right\partsBody_assemb_-_Leg_assembly_b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; visual mesh filename=body_parts\leg_back_right\partsBody_assemb_-_Leg_assembly_b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
- link fibula_top_right: geometry collision mesh filename=new_body_parts\V0Body_assemb_-_Leg_assembly_top_right-1_Fib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; visual mesh filename=new_body_parts\V0Body_assemb_-_Leg_assembly_top_right-1_Fib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
- link hip_down_right: geometry collision mesh filename=body_parts\leg_back_right\partsBody_assemb_-_Leg_assembly_b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; visual mesh filename=body_parts\leg_back_right\partsBody_assemb_-_Leg_assembly_b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
- link hip_top_right: geometry collision mesh filename=new_body_parts\V0Body_assemb_-_Leg_assembly_top_right-1_ser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; visual mesh filename=new_body_parts\V0Body_assemb_-_Leg_assembly_top_right-1_ser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
- link servo_extension_horn_mock_1_top_right: geometry collision mesh filename=; visual mesh filename=
- link servo_extension_horn_mock_2_down_right: geometry collision mesh filename=; visual mesh filename=
- link small_link_down_rigth: geometry collision mesh filename=body_parts\leg_back_right\partsBody_assemb_-_Leg_assembly_b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; visual mesh filename=body_parts\leg_back_right\partsBody_assemb_-_Leg_assembly_b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
- link tibia_down_right: geometry collision mesh filename=body_parts\leg_back_right\partsBody_assemb_-_Leg_assembly_b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; visual mesh filename=body_parts\leg_back_right\partsBody_assemb_-_Leg_assembly_b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
Joints:
- removed joint fibula_on_servo_extend_mock_2
- joint fibula_on_hip_top_right: axis 0 1 0 -> 0 0 1; origin xyz=0 0 0 rpy=0 0 0 -> xyz=-40 -50 30 rpy=0 0 0
- joint hip_down_right_on_body: axis (none) -> 1 0 0; limit (none) -> lower=0 upper=1 effort=100 velocity=0
- joint hip_top_right_on_body: limit lower=0 upper=1 effort=1 velocity=1 -> lower=0 upper=1.57 effort=1 velocity=1; origin xyz=0 0 0 rpy=0 0 0 -> xyz=170 17 100 rpy=0 0 0

Commit message: Update URDF: Change joint type to fixed and adjust limits for hip joints

File: connected_bot.urdf (robot description, URDF)
Before this commit: robot leg_design_simplified, 31 links, 16 joints
Joints:
- joint hip_top_left_on_body: axis 0 1 0 -> 1 0 0
- joint hip_top_right_on_body: limit lower=0 upper=1 effort=1 velocity=1 -> lower=-10 upper=10 effort=1 velocity=1; type revolute -> fixed
