Commit message: Update URDF: Refactor leg segments and add ankle joints for front legs

File: tesbot.urdf (robot description, URDF)
Before this commit: robot simple_quadruped, 9 links, 8 joints
Links:
- removed link leg_fl
- removed link leg_fr
- removed link leg_rl
- removed link leg_rr
- added link lower_leg_fl, mass 0.1; collision cylinder length=0.1 radius=0.02; visual cylinder length=0.1 radius=0.02
- added link lower_leg_fr, mass 0.1; collision cylinder length=0.1 radius=0.02; visual cylinder length=0.1 radius=0.02
- added link lower_leg_rl, mass 0.1; collision cylinder length=0.1 radius=0.02; visual cylinder length=0.1 radius=0.02
- added link lower_leg_rr, mass 0.1; collision cylinder length=0.1 radius=0.02; visual cylinder length=0.1 radius=0.02
- added link upper_leg_fl, mass 0.1; collision cylinder length=0.1 radius=0.02; visual cylinder length=0.1 radius=0.02
- added link upper_leg_fr, mass 0.1; collision cylinder length=0.1 radius=0.02; visual cylinder length=0.1 radius=0.02
- added link upper_leg_rl, mass 0.1; collision cylinder length=0.1 radius=0.02; visual cylinder length=0.1 radius=0.02
- added link upper_leg_rr, mass 0.1; collision cylinder length=0.1 radius=0.02; visual cylinder length=0.1 radius=0.02
Joints:
- added joint ankle_joint_fl: type revolute, parent upper_leg_fl, child lower_leg_fl, origin xyz=0 0 -0.1, axis 0 1 0, limit lower=-1.57 upper=1.57 effort=1 velocity=1
- added joint ankle_joint_fr: type revolute, parent upper_leg_fr, child lower_leg_fr, origin xyz=0 0 -0.1, axis 0 1 0, limit lower=-1.57 upper=1.57 effort=1 velocity=1
- added joint ankle_joint_rl: type revolute, parent upper_leg_rl, child lower_leg_rl, origin xyz=0 0 -0.1, axis 0 1 0, limit lower=-1.57 upper=1.57 effort=1 velocity=1
- added joint ankle_joint_rr: type revolute, parent upper_leg_rr, child lower_leg_rr, origin xyz=0 0 -0.1, axis 0 1 0, limit lower=-1.57 upper=1.57 effort=1 velocity=1
- joint knee_joint_fl: child leg_fl -> upper_leg_fl
- joint knee_joint_fr: child leg_fr -> upper_leg_fr
- joint knee_joint_rl: child leg_rl -> upper_leg_rl
- joint knee_joint_rr: child leg_rr -> upper_leg_rr
